Commit message: modified inertia

File: asset/pid_motor/urdf/pid_motor.urdf (robot description, URDF)
Before this commit: robot pid_motor, 2 links, 1 joints
Links:
- link base_link: mass 1.43119045038721 -> 0.4542
- link link1: mass 0.0152768682810347 -> 0.00978
Joints:
- joint joint1: origin xyz=0.0154890559226487 0 0.055500000000006 rpy=0 0 0 -> xyz=0.015489 0 0.0555 rpy=0 0 0
